File: pcb/pcb.kicad_sch (KiCad schematic)
At the start: 21 parts, among them J1 USB_C_Receptacle_USB2.0_14P, U1 RP2040, U2 NCP1117-3.3_TO252

Commit message: remove MCU
Parts:
- removed C1: 1uf, symbol Device:C
- removed C10, C11: 100nF, symbol Device:C
- removed C12, C13: 10uF, symbol Device:C
- removed C2, C3, C4, C5, C6, C7, C8: 100nf, symbol Device:C
- removed C9: 1uF, symbol Device:C
- removed D1: D_Schottky, symbol Device:D_Schottky
- removed J1: USB_C_Receptacle_USB2.0_14P, symbol Connector:USB_C_Receptacle_USB2.0_14P
- removed R1, R2: 5.1K, symbol Device:R
- removed R3, R4: 27, symbol Device:R
- removed U1: RP2040, Package_DFN_QFN:QFN-56-1EP_7x7mm_P0.4mm_EP3.2x3.2mm, symbol MCU_RaspberryPi:RP2040
- removed U2: NCP1117-3.3_TO252, Package_TO_SOT_SMD:TO-252-2, symbol Regulator_Linear:NCP1117-3.3_TO252
Other:
- note removed: "I need to add some symbol going to the battery"

Commit message: add TCA
Parts:
- added R? (x2): 4.7K, symbol Device:R
- added R?: 10K, symbol Device:R
- added U?: TCA9548APWR, Package_SO:TSSOP-24_4.4x7.8mm_P0.65mm, symbol Interface_Expansion:TCA9548APWR
Connections:
- new net +3V3: R?.1, R?.1, R?.1, U?.24 (VCC)
- new net GND: U?.12 (GND)
- new net SCL: R?.2, U?.22 (SCL)
- new net SDA: R?.2, U?.23 (SDA)
- new net TCARST: R?.2, U?.3 (~{RESET})
